Commit message: Correcting urdf

File: model/end_effector.urdf.xacro (robot description, xacro)
@@ -12,7 +12,7 @@
   <xacro:macro name="end_effector_kuka_lwr" params="parent name *origin">
     <joint name="sensor_joint" type="fixed">
-      <origin xyz="0 0 0" rpy="0 0 0"/>
+      <xacro:insert_block name="origin"/>
+      <child link="end_effector"/>
       <parent link="${name}_7_link"/>
-      <child link="end_effector"/>
     </joint>
     <link name="end_effector">

Commit message: -remove the material tag from the end effector link -add missing dependencies in CMakeLists.txt and package.xml -launch controller_switcher at startup in single_lwr.launch -change the path where the generated workbench xacro is saved

File: model/end_effector.urdf.xacro (robot description, xacro)
@@ -34,5 +34,4 @@
           <sphere radius="0.01" />
         </geometry>
-      <material name="Red"/>
       </visual>
       <collision>
